File: localhost/Mini_projet_BT_LCD/Mini_projet_BT_LCD.kicad_pcb (KiCad board)
At the start: 2 copper layers, 40 parts

Commit message: Mise à jour 2
Parts:
- moved TP2 3.24 mm to (146.5, 93.5)
- moved TP1 2.00 mm to (160.6, 94.0)
Connections:
- LCD1 pad 15: Net-(LCD1-A) -> Net-(A1-+5V)
- LCD1 pad 2: Net-(LCD1-VDD) -> Net-(LCD1-K)
- RV1 pad 1: Net-(LCD1-VDD) -> Net-(LCD1-K)
- TP1 pad 1: Net-(LCD1-A) -> Net-(A1-+5V)
- TP4 pad 1: Net-(LCD1-VDD) -> Net-(LCD1-K)
Routing:
- net Net-(LCD1-K): track 20.4 -> 77.0 mm, vias 0 -> 2
- net Net-(LCD1-VDD): track 47.9 -> 0.00 mm
- net Net-(A1-+5V): track 71.6 -> 103.1 mm, vias 0 -> 2
- net Net-(A1-D5): track 60.5 -> 39.1 mm
- net Net-(A1-D3): track 23.6 -> 37.9 mm
- net Net-(LCD1-A): track 11.6 -> 0.00 mm
- net Net-(A1-D2): track 30.2 -> 21.5 mm, vias 0 -> 2
- net Net-(LCD1-VO): track 30.9 -> 35.1 mm, vias 0 -> 2
